Commit message: Rebuild the platform URDF file

File: ros_unity_test/Assets/URDF/dashgobase_ao1.urdf (robot description, URDF)
Before this commit: robot box_robot, 5 links, 4 joints
Links:
- link base_link: mass 1.3729096e+00 -> 40
Joints:
- joint base_l_wheel_joint: origin xyz=0.0 0.18 -0.08 rpy=1.5707963 0 0 -> xyz=0.0 0.18 -0.08 rpy=-1.5707963 0 0
