Commit message: Control the mobile platform from ROS teleop_twist_keyboard

File: ros_unity_test/Assets/URDF/mobile_platform.urdf (robot description, URDF)
Before this commit: robot mobile_platform, 7 links, 6 joints
Links:
- removed link base_auxiliary_wheel_1_link
- removed link base_auxiliary_wheel_2_link
- removed link base_auxiliary_wheel_3_link
- removed link base_auxiliary_wheel_4_link
- added link base_back_wheel_link; collision sphere radius=0.03
- added link base_front_wheel_link; collision sphere radius=0.03
- added link laser; visual box size=0.05 0.05 0.05
- link base_left_wheel_link: geometry collision cylinder length=0.05 radius=0.06; visual cylinder length=0.05 radius=0.06
- link base_right_wheel_link: geometry collision cylinder length=0.05 radius=0.06; visual cylinder length=0.05 radius=0.06
Joints:
- removed joint auxiliary_wheel_1
- removed joint auxiliary_wheel_2
- removed joint auxiliary_wheel_3
- removed joint auxiliary_wheel_4
- removed joint left_right_joint
- added joint back_wheel: type fixed, parent base_link, child base_back_wheel_link, origin xyz=-0.35 0 -0.03 rpy=0 0 0
- added joint front_wheel: type fixed, parent base_link, child base_front_wheel_link, origin xyz=0 0 -0.03 rpy=0 0 0
- added joint right_wheel_joint: type continuous, parent base_link, child base_right_wheel_link, origin xyz=-0.2 -0.15 0 rpy=-1.5707963 0 0, axis 0 0 1, limit effort=100 velocity=100
- added joint top_t_laser: type fixed, parent base_link, child laser, origin xyz=-0.05 0 0.16 rpy=0 0 0
- joint left_wheel_joint: origin xyz=0.01 0.15 0.05 rpy=0 1.5707 0 -> xyz=-0.2 0.15 0 rpy=-1.5707963 0 0
