Commit message: Modify the URDF of platform and kinovaMsg class name

File: ros_unity_test/Assets/URDF/mobile_manipulator.urdf (robot description, URDF)
Before this commit: robot mobile_manipulator, 30 links, 29 joints
Links:
- removed link platform_link
- added link base_platform, mass 36; collision mesh filename=package://platform_description/meshes/platform.STL scale=0.001 0.001 0.001; visual mesh filename=package://platform_description/meshes/platform.STL scale=0.001 0.001 0.001
Joints:
- joint back_wheel: origin xyz=-0.35 0 -0.03 rpy=0 0 0 -> xyz=-0.15 0 -0.025 rpy=0 0 0; parent platform_link -> base_platform
- joint front_wheel: origin xyz=0 0 -0.03 rpy=0 0 0 -> xyz=0.15 0 -0.025 rpy=0 0 0; parent platform_link -> base_platform
- joint left_wheel_joint: origin xyz=-0.2 0.15 0 rpy=-1.5707963 0 0 -> xyz=0 0.15 0 rpy=-1.5707963 0 0; parent platform_link -> base_platform
- joint platform_arm_link: origin xyz=-0.21 0 0.33 rpy=0 0 0 -> xyz=0 0 0.34 rpy=0 0 0; parent platform_link -> base_platform
- joint right_wheel_joint: origin xyz=-0.2 -0.15 0 rpy=-1.5707963 0 0 -> xyz=0 -0.15 0 rpy=-1.5707963 0 0; parent platform_link -> base_platform
- joint top_t_laser: origin xyz=-0.05 0 0.16 rpy=0 0 0 -> xyz=0.15 0 0.16 rpy=0 0 0; parent platform_link -> base_platform

File: ros_unity_test/Assets/URDF/mobile_platform.urdf (robot description, URDF)
Before this commit: robot mobile_platform, 6 links, 5 joints
Links:
- removed link base_link
- added link base_platform, mass 36; collision mesh filename=package://platform_description/meshes/platform.STL scale=0.001 0.001 0.001; visual mesh filename=package://platform_description/meshes/platform.STL scale=0.001 0.001 0.001
Joints:
- joint back_wheel: origin xyz=-0.35 0 -0.03 rpy=0 0 0 -> xyz=-0.15 0 -0.025 rpy=0 0 0; parent base_link -> base_platform
- joint front_wheel: origin xyz=0 0 -0.03 rpy=0 0 0 -> xyz=0.15 0 -0.025 rpy=0 0 0; parent base_link -> base_platform
- joint left_wheel_joint: origin xyz=-0.2 0.15 0 rpy=-1.5707963 0 0 -> xyz=0 0.15 0 rpy=-1.5707963 0 0; parent base_link -> base_platform
- joint right_wheel_joint: origin xyz=-0.2 -0.15 0 rpy=-1.5707963 0 0 -> xyz=0 -0.15 0 rpy=-1.5707963 0 0; parent base_link -> base_platform
- joint top_t_laser: origin xyz=-0.05 0 0.16 rpy=0 0 0 -> xyz=0.15 0 0.16 rpy=0 0 0; parent base_link -> base_platform
